Commit message: sim size fix and para fix

File: student_ws/src/rb3302_simulation/models/simulated_waverover/model.urdf (robot description, URDF)
Before this commit: robot waverover, 2 links, 1 joints
Links:
- added link left_wheel_visual; visual cylinder length=0.03 radius=0.035
- added link right_wheel_visual; visual cylinder length=0.03 radius=0.035
- link base_link: geometry visual box size=0.19 0.11 0.10
Joints:
- added joint left_wheel_visual_joint: type fixed, parent base_link, child left_wheel_visual, origin xyz=0 0.07 0 rpy=0 0 0
- added joint right_wheel_visual_joint: type fixed, parent base_link, child right_wheel_visual, origin xyz=0 -0.07 0 rpy=0 0 0
